Commit message: AMCL Workgin
odom is now showing in rvis and I am able to adjust robot parameters.

File: catkin_ws/src/udacity_bot/urdf/my_robot.xacro (robot description, xacro)
@@ -2,5 +2,5 @@
 <!-- Robot Base -->
 <robot name="my_robot" xmlns:xacro="http://www.ros.org/wiki/xacro">
-<xacro:include filename="$(find my_robot)/urdf/my_robot.gazebo" />
+<xacro:include filename="$(find udacity_bot)/urdf/my_robot.gazebo" />
   <link name="robot_footprint"></link>
   <joint name="robot_footprint_joint" type="fixed">
@@ -235,5 +235,5 @@
       <origin xyz="0.0 0.0 0.0" rpy="0.0 0.0 0.0"/>
       <geometry>
-        <mesh filename="package://my_robot/meshes/hokuyo.dae"/>
+        <mesh filename="package://udacity_bot/meshes/hokuyo.dae"/>
       </geometry>
     </visual>

Commit message: Update my_robot.xacro
Removed 2nd set of wheels to make robot act like the original version.

File: catkin_ws/src/udacity_bot/urdf/my_robot.xacro (robot description, xacro)
@@ -82,5 +82,5 @@
   </link>
   <joint type="continuous" name="left_wheel_hinge">
-    <origin xyz="0.2 0.15 0" rpy="0 0 0"/>
+    <origin xyz="0.0 0.15 0" rpy="0 0 0"/>
     <child link="left_wheel"/>
     <parent link="chassis"/>
@@ -113,5 +113,5 @@
   </link>
   <joint type="continuous" name="right_wheel_hinge">
-    <origin xyz="0.2 -0.15 0" rpy="0 0 0"/>
+    <origin xyz="0.0 -0.15 0" rpy="0 0 0"/>
     <child link="right_wheel"/>
     <parent link="chassis"/>
@@ -121,66 +121,4 @@
   </joint>
   <!-- Second Set of Wheels -->
-  <link name='left2_wheel'>
-    <inertial>
-      <mass value="5.0"/>
-      <origin xyz="0.0 0.0 0.0" rpy="0.0 1.5707 1.5707"/>
-      <inertia
-          ixx="0.1" ixy="0" ixz="0"
-          iyy="0.1" iyz="0"
-          izz="0.1"
-      />
-    </inertial>
-    <collision name='left2_wheel_collision'>
-      <origin xyz="0.0 0.0 0.0" rpy="0.0 1.5707 1.5707"/>
-      <geometry>
-        <cylinder length="0.05" radius="0.1"/>
-      </geometry>
-    </collision>
-    <visual name='left2_wheel_visual'>
-      <origin xyz="0.0 0.0 0.0" rpy="0.0 1.5707 1.5707"/>
-      <geometry>
-        <cylinder length="0.05" radius="0.1"/>
-      </geometry>
-    </visual>
-  </link>
-  <joint type="continuous" name="left2_wheel_hinge">
-    <origin xyz="-0.25 0.15 0" rpy="0 0 0"/>
-    <child link="left2_wheel"/>
-    <parent link="chassis"/>
-    <axis xyz="0 1 0" rpy="0 0 0"/>
-    <limit effort="10000" velocity="1000"/>
-    <dynamics damping="1.0" friction="1.0"/>
-  </joint>
-  <link name='right2_wheel'>
-    <inertial>
-      <mass value="5.0"/>
-      <origin xyz="0.0 0.0 0.0" rpy="0.0 1.5707 1.5707"/>
-      <inertia
-          ixx="0.1" ixy="0" ixz="0"
-          iyy="0.1" iyz="0"
-          izz="0.1"
-      />
-    </inertial>
-    <collision name='right2_wheel_collision'>
-      <origin xyz="0.0 0.0 0.0" rpy="0.0 1.5707 1.5707"/>
-      <geometry>
-        <cylinder length="0.05" radius="0.1"/>
-      </geometry>
-    </collision>
-    <visual name='right2_wheel_visual'>
-      <origin xyz="0.0 0.0 0.0" rpy="0.0 1.5707 1.5707"/>
-      <geometry>
-        <cylinder length="0.05" radius="0.1"/>
-      </geometry>
-    </visual>
-  </link>
-  <joint type="continuous" name="right2_wheel_hinge">
-    <origin xyz="-0.25 -0.15 0" rpy="0 0 0"/>
-    <child link="right2_wheel"/>
-    <parent link="chassis"/>
-    <axis xyz="0 1 0" rpy="0 0 0"/>
-    <limit effort="10000" velocity="1000"/>
-    <dynamics damping="1.0" friction="1.0"/>
-  </joint>
   <!-- Peripherals -->
   <link name='camera'>

Commit message: Finalization
Robot is able to localize using 2D nav goal in RVIz.
Removing extraneous files

File: catkin_ws/src/udacity_bot/urdf/my_robot.xacro (robot description, xacro)
@@ -23,5 +23,5 @@
       <origin xyz="0 0 0" rpy=" 0 0 0"/>
       <geometry>
-        <box size=".5 .2 .1"/>
+        <box size=".4 .2 .1"/>
       </geometry>
     </collision>
@@ -29,5 +29,5 @@
       <origin xyz="0 0 0" rpy=" 0 0 0"/>
       <geometry>
-        <box size=".5 .2 .1"/>
+        <box size=".4 .2 .1"/>
       </geometry>
     </visual>
